File: schematic/5x5_LED_Cube/5x5_LED_Cube_Driver.kicad_pcb (KiCad board)
At the start: 2 copper layers, 88.9 x 81.3 mm, 46 parts, among them J1 Arduino, J2 Power, J3 Layers, Q1 DMG2305UX, Q2 DMG2305UX, Q3 DMG2305UX, Q4 DMG2305UX, Q5 DMG2305UX, U1 TLC5940NT, U2 TLC5940NT

Commit message: Updated schematic and footprints
Other:
- net class Default removed
